File: ICB8xduino-328p.kicad_pcb (KiCad board)
At the start: 2 copper layers, 73.7 x 48.3 mm, 35 parts, among them J1 BARREL_JACK, J2 Serial, J4 AE-FT234X, SW1 RESET, U1 TM78M05F, U2 ATMEGA328-PU, Y1 16MHz

Commit message: 個別ライブラリをプロジェクトに入れた
Parts:
- SW1: footprint abtc:SW_PUSH_Single_6mm -> ICB8xduino:SW_PUSH_Single_6mm
- U1: value TM78M05F -> TA78M05F
- Y1: footprint abtc:Resonator__HC49-U_Vertical -> ICB8xduino:Resonator__HC49-U_Vertical
Other:
- board text removed: "ICB8xduino -328P"
Changed lines of the file:
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@@
     (links 90)
     (no_connects 0)
-    (area 69.454047 31.59 198.35 85.165001)
+    (area 110.414999 36.754999 184.225001 85.165001)
     (thickness 1.6)
-    (drawings 72)
+    (drawings 70)
     (tracks 508)
     (zones 0)
@@
     )
   )
-  (module abtc:SW_PUSH_Single_6mm (layer F.Cu)
-    (at 182.88 57.15 180)
-    (descr https://www.omron.com/ecb/products/pdf/en-b3f.pdf)
-    (tags "tact sw push 6mm")
-    (fp_text reference SW1 (at 3.81 0 180) (layer F.SilkS)
-      (effects (font (size 1 1) (thickness 0.15)))
-    )
-    (fp_text value RESET (at 10.16 0 180) (layer F.Fab)
-      (effects (font (size 1 1) (thickness 0.15)))
-    )
-    (fp_line (start 3.25 -1.75) (end 6.25 -1.75) (layer F.Fab) (width 0.1))
-    (fp_line (start 6.25 -1.75) (end 6.25 1.75) (layer F.Fab) (width 0.1))
-    (fp_line (start 6.25 1.75) (end 0.25 1.75) (layer F.Fab) (width 0.1))
-    (fp_line (start 0.25 1.75) (end 0.25 -1.75) (layer F.Fab) (width 0.1))
-    (fp_line (start 0.25 -1.75) (end 3.25 -1.75) (layer F.Fab) (width 0.1))
-    (fp_line (start 7.75 -1.881) (end 8 -1.881) (layer F.CrtYd) (width 0.05))
-    (fp_line (start 8 -1.5) (end 8 -1.25) (layer F.CrtYd) (width 0.05))
-    (fp_line (start -1.5 -1.25) (end -1.5 -1.5) (layer F.CrtYd) (width 0.05))
-    (fp_line (start -1.5 -1.881) (end -1.25 -1.881) (layer F.CrtYd) (width 0.05))
-    (fp_line (start -1.25 -1.881) (end 7.75 -1.881) (layer F.CrtYd) (width 0.05))
-    (fp_line (start -1.5 2.1392) (end -1.5 -1.885) (layer F.CrtYd) (width 0.05))
-    (fp_line (start 8 2.1392) (end -1.4786 2.1392) (layer F.CrtYd) (width 0.05))
-    (fp_line (start 8 -1.885) (end 8 2.1392) (layer F.CrtYd) (width 0.05))
-    (fp_line (start 1 2) (end 5.5 2) (layer F.SilkS) (width 0.12))
-    (fp_line (start 5.5 -2) (end 1 -2) (layer F.SilkS) (width 0.12))
-    (pad 1 thru_hole circle (at 0 0 270) (size 2.1 2.1) (drill 1.2) (layers *.Cu *.Mask)
-      (net 31 GNDD))
-    (pad 2 thru_hole circle (at 6.5 0 270) (size 2.1 2.1) (drill 1.2) (layers *.Cu *.Mask)
-      (net 7 /RESET))
-    (model ${KISYS3DMOD}/Buttons_Switches_THT.3dshapes/SW_PUSH_6mm.wrl
-      (at (xyz 0.005 0 0))
-      (scale (xyz 0.3937 0.3937 0.3937))
-      (rotate (xyz 0 0 0))
-    )
-  )
   (module TO_SOT_Packages_THT:SIPAK-1EP_Horizontal (layer F.Cu)
     (at 136.144 45.974 270)
@@
       (effects (font (size 1 1) (thickness 0.15)))
     )
-    (fp_text value TM78M05F (at 2.286 1.9 270) (layer F.Fab)
+    (fp_text value TA78M05F (at 2.286 1.9 270) (layer F.Fab)
       (effects (font (size 1 1) (thickness 0.15)))
     )
@@
       (at (xyz 0 0 0))
       (scale (xyz 1 1 1))
-      (rotate (xyz 0 0 0))
-    )
-  )
-  (module abtc:Resonator__HC49-U_Vertical (layer F.Cu)
-    (at 153.162 57.658 180)
-    (descr "Crystal THT HC-49/U http://5hertz.com/pdfs/04404_D.pdf")
-    (tags "THT crystalHC-49/U")
-    (fp_text reference Y1 (at 2.54 -1.651 180) (layer F.SilkS)
-      (effects (font (size 1 1) (thickness 0.15)))
-    )
-    (fp_text value 16MHz (at 2.44 3.525 180) (layer F.Fab)
-      (effects (font (size 1 1) (thickness 0.15)))
-    )
-    (fp_arc (start -0.685 0) (end -0.685 -2.325) (angle -180) (layer F.Fab) (width 0.1))
-    (fp_arc (start 5.565 0) (end 5.565 -2.325) (angle 180) (layer F.Fab) (width 0.1))
-    (fp_arc (start -0.56 0) (end -0.56 -2) (angle -180) (layer F.Fab) (width 0.1))
-    (fp_arc (start 5.44 0) (end 5.44 -2) (angle 180) (layer F.Fab) (width 0.1))
-    (fp_arc (start -0.685 0) (end -0.685 -2.525) (angle -180) (layer F.SilkS) (width 0.12))
-    (fp_arc (start 5.565 0) (end 5.565 -2.525) (angle 180) (layer F.SilkS) (width 0.12))
-    (fp_line (start -0.685 -2.325) (end 5.565 -2.325) (layer F.Fab) (width 0.1))
-    (fp_line (start -0.685 2.325) (end 5.565 2.325) (layer F.Fab) (width 0.1))
-    (fp_line (start -0.56 -2) (end 5.44 -2) (layer F.Fab) (width 0.1))
-    (fp_line (start -0.56 2) (end 5.44 2) (layer F.Fab) (width 0.1))
-    (fp_line (start -0.685 -2.525) (end 5.565 -2.525) (layer F.SilkS) (width 0.12))
-    (fp_line (start -0.685 2.525) (end 5.565 2.525) (layer F.SilkS) (width 0.12))
-    (fp_line (start -3.5 -2.8) (end -3.5 2.8) (layer F.CrtYd) (width 0.05))
-    (fp_line (start -3.5 2.8) (end 8.4 2.8) (layer F.CrtYd) (width 0.05))
-    (fp_line (start 8.4 2.8) (end 8.4 -2.8) (layer F.CrtYd) (width 0.05))
-    (fp_line (start 8.4 -2.8) (end -3.5 -2.8) (layer F.CrtYd) (width 0.05))
-    (pad 2 thru_hole circle (at 2.44 0 180) (size 1.5 1.5) (drill 0.8) (layers *.Cu *.Mask)
-      (net 31 GNDD))
-    (pad 1 thru_hole circle (at 0 0 180) (size 1.5 1.5) (drill 0.8) (layers *.Cu *.Mask)
-      (net 4 /XTAL1))
-    (pad 3 thru_hole circle (at 4.88 0 180) (size 1.5 1.5) (drill 0.8) (layers *.Cu *.Mask)
-      (net 5 /XTAL2))
-    (model Crystals.3dshapes/Crystal_HC49-U_Vertical.wrl
-      (at (xyz 0 0 0))
-      (scale (xyz 0.393701 0.393701 0.393701))
       (rotate (xyz 0 0 0))
     )
@@
     (pad "" np_thru_hole circle (at 0 0) (size 3.7 3.7) (drill 3.6) (layers *.Cu *.Mask))
   )
+  (module ICB8xduino:SW_PUSH_Single_6mm (layer F.Cu)
+    (at 182.88 57.15 180)
+    (descr https://www.omron.com/ecb/products/pdf/en-b3f.pdf)
+    (tags "tact sw push 6mm")
+    (fp_text reference SW1 (at 3.429 -2.794 180) (layer F.SilkS)
+      (effects (font (size 1 1) (thickness 0.15)))
+    )
+    (fp_text value RESET (at 10.16 0 180) (layer F.Fab)
+      (effects (font (size 1 1) (thickness 0.15)))
+    )
+    (fp_text user %R (at 3.175 0.127 180) (layer F.Fab)
+      (effects (font (size 1 1) (thickness 0.15)))
+    )
+    (fp_line (start 3.25 -1.75) (end 6.25 -1.75) (layer F.Fab) (width 0.1))
+    (fp_line (start 6.25 -1.75) (end 6.25 1.75) (layer F.Fab) (width 0.1))
+    (fp_line (start 6.25 1.75) (end 0.25 1.75) (layer F.Fab) (width 0.1))
+    (fp_line (start 0.25 1.75) (end 0.25 -1.75) (layer F.Fab) (width 0.1))
+    (fp_line (start 0.25 -1.75) (end 3.25 -1.75) (layer F.Fab) (width 0.1))
+    (fp_line (start 7.75 -1.881) (end 8 -1.881) (layer F.CrtYd) (width 0.05))
+    (fp_line (start 8 -1.5) (end 8 -1.25) (layer F.CrtYd) (width 0.05))
+    (fp_line (start -1.5 -1.25) (end -1.5 -1.5) (layer F.CrtYd) (width 0.05))
+    (fp_line (start -1.5 -1.881) (end -1.25 -1.881) (layer F.CrtYd) (width 0.05))
+    (fp_line (start -1.25 -1.881) (end 7.75 -1.881) (layer F.CrtYd) (width 0.05))
+    (fp_line (start -1.5 2.1392) (end -1.5 -1.885) (layer F.CrtYd) (width 0.05))
+    (fp_line (start 8 2.1392) (end -1.4786 2.1392) (layer F.CrtYd) (width 0.05))
+    (fp_line (start 8 -1.885) (end 8 2.1392) (layer F.CrtYd) (width 0.05))
+    (fp_line (start 1 2) (end 5.5 2) (layer F.SilkS) (width 0.12))
+    (fp_line (start 5.5 -2) (end 1 -2) (layer F.SilkS) (width 0.12))
+    (pad 1 thru_hole circle (at 0 0 270) (size 2.1 2.1) (drill 1.2) (layers *.Cu *.Mask)
+      (net 31 GNDD))
+    (pad 2 thru_hole circle (at 6.5 0 270) (size 2.1 2.1) (drill 1.2) (layers *.Cu *.Mask)
+      (net 7 /RESET))
+    (model ${KISYS3DMOD}/Buttons_Switches_THT.3dshapes/SW_PUSH_6mm.wrl
+      (at (xyz 0.005 0 0))
+      (scale (xyz 0.3937 0.3937 0.3937))
+      (rotate (xyz 0 0 0))
+    )
+  )
+  (module ICB8xduino:Resonator__HC49-U_Vertical (layer F.Cu)
+    (at 153.162 57.658 180)
+    (descr "Crystal THT HC-49/U http://5hertz.com/pdfs/04404_D.pdf")
+    (tags "THT crystalHC-49/U")
+    (fp_text reference Y1 (at 2.44 -3.525 180) (layer F.SilkS)
+      (effects (font (size 1 1) (thickness 0.15)))
+    )
+    (fp_text value 16MHz (at 2.44 3.525 180) (layer F.Fab)
+      (effects (font (size 1 1) (thickness 0.15)))
+    )
+    (fp_arc (start -0.685 0) (end -0.685 -2.325) (angle -180) (layer F.Fab) (width 0.1))
+    (fp_arc (start 5.565 0) (end 5.565 -2.325) (angle 180) (layer F.Fab) (width 0.1))
+    (fp_arc (start -0.56 0) (end -0.56 -2) (angle -180) (layer F.Fab) (width 0.1))
+    (fp_arc (start 5.44 0) (end 5.44 -2) (angle 180) (layer F.Fab) (width 0.1))
+    (fp_arc (start -0.685 0) (end -0.685 -2.525) (angle -180) (layer F.SilkS) (width 0.12))
+    (fp_arc (start 5.565 0) (end 5.565 -2.525) (angle 180) (layer F.SilkS) (width 0.12))
+    (fp_line (start -0.685 -2.325) (end 5.565 -2.325) (layer F.Fab) (width 0.1))
+    (fp_line (start -0.685 2.325) (end 5.565 2.325) (layer F.Fab) (width 0.1))
+    (fp_line (start -0.56 -2) (end 5.44 -2) (layer F.Fab) (width 0.1))
+    (fp_line (start -0.56 2) (end 5.44 2) (layer F.Fab) (width 0.1))
+    (fp_line (start -0.685 -2.525) (end 5.565 -2.525) (layer F.SilkS) (width 0.12))
+    (fp_line (start -0.685 2.525) (end 5.565 2.525) (layer F.SilkS) (width 0.12))
+    (fp_line (start -3.5 -2.8) (end -3.5 2.8) (layer F.CrtYd) (width 0.05))
+    (fp_line (start -3.5 2.8) (end 8.4 2.8) (layer F.CrtYd) (width 0.05))
+    (fp_line (start 8.4 2.8) (end 8.4 -2.8) (layer F.CrtYd) (width 0.05))
+    (fp_line (start 8.4 -2.8) (end -3.5 -2.8) (layer F.CrtYd) (width 0.05))
+    (pad 2 thru_hole circle (at 2.44 0 180) (size 1.5 1.5) (drill 0.8) (layers *.Cu *.Mask)
+      (net 31 GNDD))
+    (pad 1 thru_hole circle (at 0 0 180) (size 1.5 1.5) (drill 0.8) (layers *.Cu *.Mask)
+      (net 4 /XTAL1))
+    (pad 3 thru_hole circle (at 4.88 0 180) (size 1.5 1.5) (drill 0.8) (layers *.Cu *.Mask)
+      (net 5 /XTAL2))
+    (model Crystals.3dshapes/Crystal_HC49-U_Vertical.wrl
+      (at (xyz 0 0 0))
+      (scale (xyz 0.393701 0.393701 0.393701))
+      (rotate (xyz 0 0 0))
+    )
+  )
   (gr_text RESET (at 179.578 60.071) (layer F.SilkS)
     (effects (font (size 1 1) (thickness 0.1)))
@@
     (effects (font (size 1 1) (thickness 0.1)))
   )
-  (gr_text "(C)Toshio Abe,2017" (at 76.835 71.755) (layer B.Cu)
-    (effects (font (size 1 1) (thickness 0.2)) (justify mirror))
-  )
-  (gr_text "ICB8xduino\n-328P" (at 85.725 73.025) (layer B.Cu)
-    (effects (font (size 1.5 1.5) (thickness 0.2)) (justify right mirror))
-  )
   (gr_text "(C)Toshio Abe,2017" (at 146.685 83.185) (layer F.SilkS)
